Commit message: Update gp8_macro.xacro

File: motoman_gp8_support/urdf/gp8_macro.xacro (robot description, xacro)
@@ -187,12 +187,4 @@
         <child link="${prefix}tool0"/>
     </joint>
-    <!-- end of joint list -->
-    <!-- ROS base_link to Robot Manufacturer World Coordinates transform -->
-    <link name="${prefix}base" />
-    <joint name="${prefix}base_link-base" type="fixed">
-        <origin xyz="0 0 0" rpy="0 0 0"/>
-        <parent link="${prefix}base_rail"/>
-        <child link="${prefix}base"/>
-    </joint>
     </xacro:macro>
 </robot>
